File: rev_b/bus_bridge_encoders_sonar.kicad_pcb (KiCad board)
At the start: 2 copper layers, 100 x 50 mm, 63 parts, among them J1 POWER_SELECT, J2 TERMINATE_JUMPER, SW1 MJTP1243, U1 LM2940, U2 LTV-826, U3 LTV-826, U4 LTV-826, U5 754410, U6 LM2940, U7 74HCT08, U8 MCP2562, U9 ATMEGA328_DIP28, X1 CRYSTAL

Commit message: Did first cut of revision B.
Parts:
- removed N4: ENCODER_CONNECTOR, Bus_Bridge_Encoders_Sonar_Rev_A:Pin_Header_Straight_1x04
- removed R10, R11, R12, R13, R9: 10K, Bus_Bridge_Encoders_Sonar_Rev_A:Resistor_Horizontal_400
- removed R21: 33K, Bus_Bridge_Encoders_Sonar_Rev_A:Resistor_Horizontal_400
- removed R3, R4, R5, R6, R7: 470, Bus_Bridge_Encoders_Sonar_Rev_A:Resistor_Horizontal_400
- added D2: LED, Bus_Bridge_Encoders_Sonar:T1_LED, F.Cu at (158.1, 146.1)
- C1, C3, C6, C9: footprint Bus_Bridge_Encoders_Sonar_Rev_A:Capacitor4x3RM2-5_RevB -> Bus_Bridge_Encoders_Sonar:Capacitor4x3RM2-5_RevB
- C10, C11, C12, C13, C14, C2, C4, C5, C7, C8: footprint Bus_Bridge_Encoders_Sonar_Rev_A:Capacitor3MMDiscRM2.5 -> Bus_Bridge_Encoders_Sonar:Capacitor3MMDiscRM2.5
- D1: footprint Bus_Bridge_Encoders_Sonar_Rev_A:Diode_DO-41_SOD81_Horizontal_RM10 -> Bus_Bridge_Encoders_Sonar:Diode_DO-41_SOD81_Horizontal_RM10
- G1: footprint Bus_Bridge_Encoders_Sonar_Rev_A:OSHW_LOGO_400mil -> Bus_Bridge_Encoders_Sonar:OSHW_LOGO_300mil
- H1, H2, H3, H4: footprint Bus_Bridge_Encoders_Sonar_Rev_A:MountingHole_3mm -> Bus_Bridge_Encoders_Sonar:MountingHole_3mm
- J1, J2: footprint Bus_Bridge_Encoders_Sonar_Rev_A:Pin_Header_Straight_1x03 -> Bus_Bridge_Encoders_Sonar:Pin_Header_Straight_1x03
- N1: footprint Bus_Bridge_Encoders_Sonar_Rev_A:Pin_Header_Straight_2x05_Shrouded -> Bus_Bridge_Encoders_Sonar:Pin_Header_Straight_2x05_Shrouded
- N2: footprint Bus_Bridge_Encoders_Sonar_Rev_A:Pin_Header_Straight_1x06 -> Bus_Bridge_Encoders_Sonar:Pin_Header_Straight_1x06
- N3: value ENCODER_CONNECTOR -> AVR_ISP_HEADER; footprint Bus_Bridge_Encoders_Sonar_Rev_A:Pin_Header_Straight_1x04 -> Bus_Bridge_Encoders_Sonar:Pin_Header_Straight_2x03
- N5, N6: value MOTOR_CONNECTOR -> MOTOR_ENCODER_CONN; footprint Bus_Bridge_Encoders_Sonar_Rev_A:Pin_Header_Straight_1x02 -> Bus_Bridge_Encoders_Sonar:Pin_Header_Straight_2x04_Shrouded
- N7, N8: footprint Bus_Bridge_Encoders_Sonar_Rev_A:Pin_Header_Straight_1x04 -> Bus_Bridge_Encoders_Sonar:Pin_Header_Straight_1x04
- R1, R14, R15, R16, R19, R22: footprint Bus_Bridge_Encoders_Sonar_Rev_A:Resistor_Horizontal_400 -> Bus_Bridge_Encoders_Sonar:Resistor_Horizontal_400
- R17, R20: value 22K -> 100K; footprint Bus_Bridge_Encoders_Sonar_Rev_A:Resistor_Horizontal_400 -> Bus_Bridge_Encoders_Sonar:Resistor_Horizontal_400
- R18: value 33K -> 100K; footprint Bus_Bridge_Encoders_Sonar_Rev_A:Resistor_Horizontal_400 -> Bus_Bridge_Encoders_Sonar:Resistor_Horizontal_400
- R2: footprint Bus_Bridge_Encoders_Sonar_Rev_A:Resistor_Horizontal_400 -> Bus_Bridge_Encoders_Sonar:DIP-16__300
- R8: footprint Bus_Bridge_Encoders_Sonar_Rev_A:Resistor_Horizontal_400 -> Bus_Bridge_Encoders_Sonar:Pin_Header_Straight_1x07
- SW1: footprint Bus_Bridge_Encoders_Sonar_Rev_A:Button_6.5MM -> Bus_Bridge_Encoders_Sonar:Button_6.5MM
- U1, U6: footprint Bus_Bridge_Encoders_Sonar_Rev_A:TO-220_Neutral123_Horizontal_LargePads -> Bus_Bridge_Encoders_Sonar:TO-220_Neutral123_Horizontal_LargePads
- U2, U3, U4, U8: footprint Bus_Bridge_Encoders_Sonar_Rev_A:DIP-8__300 -> Bus_Bridge_Encoders_Sonar:DIP-8__300
- U5: footprint Bus_Bridge_Encoders_Sonar_Rev_A:DIP-16__300 -> Bus_Bridge_Encoders_Sonar:DIP-16__300
- U7: footprint Bus_Bridge_Encoders_Sonar_Rev_A:DIP-14__300 -> Bus_Bridge_Encoders_Sonar:DIP-14__300
- U9: footprint Bus_Bridge_Encoders_Sonar_Rev_A:DIP-28__300 -> Bus_Bridge_Encoders_Sonar:DIP-28__300
- X1: value CRYSTAL -> 16MHz; footprint Bus_Bridge_Encoders_Sonar_Rev_A:Crystal_HC49-U_Vertical -> Bus_Bridge_Encoders_Sonar:Crystal_HC49-U_Vertical
- moved N6 44.2 mm to (170.2, 144.8), turned to 0 degrees
- moved R18 35.8 mm to (118.7, 141.6)
- moved R8 22.9 mm to (174.0, 130.2), turned to 90 degrees
- moved C4 20.3 mm to (194.9, 123.8)
- moved N5 19.7 mm to (181.6, 105.4), turned to 180 degrees
- moved C3 16.8 mm to (188.6, 146.7), turned to 180 degrees
- moved C1 16.4 mm to (183.5, 146.7), turned to 0 degrees
- moved J1 15.3 mm to (194.9, 131.4)
- moved U1 12.2 mm to (187.3, 142.2), turned to 0 degrees
- moved C2 12.0 mm to (181.6, 142.2), turned to 90 degrees
- moved R1 11.4 mm to (180.3, 132.1), turned to 270 degrees
- moved R2 10.3 mm to (156.2, 116.2), turned to 270 degrees
- moved N3 8.91 mm to (147.3, 145.4)
- moved U5 8.47 mm to (186.1, 115.6)
- moved U4 3.81 mm to (167.0, 132.7)
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Connections:
- C11 pad 1: +5V -> VCC
- C12 pad 1: +5V -> VCC
- C13 pad 1: +5V -> VCC
- C14 pad 1: +5V -> VCC
- C8 pad 1: +5V -> VCC
- C9 pad 1: +5V -> VCC
- D1 pad -: +5V -> VCC
- J2 pad 3: Net-(J2-Pad3) -> (no net)
- N2 pad 2: Net-(N2-Pad2) -> (no net)
- N2 pad 3: Net-(N2-Pad3) -> (no net)
- N3 pad 1: GND -> /D12
- N3 pad 2: /D5 -> VCC
- N3 pad 3: /D6 -> /D13
- N3 pad 4: +5V -> /D11
- N5 pad 1: /M1+ -> /A0
- N5 pad 2: /M1- -> GND
- N6 pad 1: /M2+ -> /D2
- N6 pad 2: /M2- -> GND
- N7 pad 2: /A1 -> /D6
- N7 pad 3: /D9 -> /D5
- N7 pad 4: +5V -> VCC
- N8 pad 2: /A0 -> /D3
- N8 pad 3: /D3 -> /D4
- N8 pad 4: +5V -> VCC
- R17 pad 2: +5V -> VCC
- R18 pad 1: GND -> Net-(R18-Pad1)
- R18 pad 2: Net-(N2-Pad4) -> VCC
- R2 pad 1: /D13 -> /D10
- R2 pad 2: Net-(R2-Pad2) -> /D12
- R20 pad 2: +5V -> VCC
- R22 pad 2: +5V -> VCC
- U2 pad 1: Net-(R2-Pad2) -> Net-(R2-Pad16)
- U2 pad 3: Net-(R3-Pad2) -> Net-(R2-Pad15)
- U2 pad 5: Net-(R9-Pad2) -> Net-(R8-Pad6)
- U2 pad 7: Net-(R8-Pad2) -> Net-(R8-Pad7)
- U3 pad 1: Net-(R4-Pad2) -> Net-(R2-Pad14)
- U3 pad 3: Net-(R5-Pad2) -> Net-(R2-Pad13)
- U3 pad 5: Net-(R11-Pad2) -> Net-(R8-Pad4)
- U3 pad 7: Net-(R10-Pad2) -> Net-(R8-Pad5)
- U4 pad 1: Net-(R6-Pad2) -> Net-(R2-Pad12)
- U4 pad 3: Net-(R7-Pad2) -> Net-(R2-Pad11)
- U4 pad 5: Net-(R13-Pad2) -> Net-(R8-Pad2)
- U4 pad 7: Net-(R12-Pad2) -> Net-(R8-Pad3)
- U5 pad 1: Net-(R9-Pad2) -> Net-(R8-Pad6)
- U5 pad 10: Net-(R11-Pad2) -> Net-(R8-Pad4)
- U5 pad 15: Net-(R13-Pad2) -> Net-(R8-Pad2)
- U5 pad 2: Net-(R8-Pad2) -> Net-(R8-Pad7)
- U5 pad 7: Net-(R10-Pad2) -> Net-(R8-Pad5)
- U5 pad 9: Net-(R12-Pad2) -> Net-(R8-Pad3)
- U6 pad 3: +5V -> VCC
- U7 pad 1: Net-(U7-Pad1) -> Net-(R18-Pad1)
- U7 pad 10: (no net) -> Net-(U7-Pad10)
- U7 pad 11: (no net) -> Net-(U7-Pad10)
- U7 pad 12: (no net) -> VCC
- U7 pad 13: (no net) -> VCC
- U7 pad 14: +5V -> VCC
- U7 pad 4: +5V -> VCC
- U7 pad 9: (no net) -> Net-(U7-Pad10)
- U8 pad 1: Net-(U7-Pad1) -> /TXD
- U8 pad 3: +5V -> VCC
- U8 pad 4: /TXD -> Net-(R18-Pad1)
- U8 pad 5: +5V -> VCC
- U9 pad 20: +5V -> VCC
- U9 pad 21: Net-(U9-Pad21) -> (no net)
- U9 pad 25: Net-(U9-Pad25) -> (no net)
- U9 pad 26: Net-(U9-Pad26) -> (no net)
- U9 pad 27: Net-(U9-Pad27) -> (no net)
- U9 pad 28: Net-(U9-Pad28) -> Net-(R2-Pad10)
- U9 pad 7: +5V -> VCC
Routing:
- net VCC: track 0.00 -> 234.3 mm, vias 0 -> 3
- net +5V: track 190.0 -> 0.00 mm, vias 3 -> 0
- net /BGND: track 228.4 -> 170.7 mm
- net /~RESET: track 41.2 -> 94.8 mm, vias 0 -> 1
- net Net-(R10-Pad2): track 51.7 -> 0.00 mm, vias 2 -> 0
- net Net-(R12-Pad2): track 46.3 -> 0.00 mm
- net Net-(R8-Pad3): track 0.00 -> 41.9 mm, vias 0 -> 2
- net GND: track 226.9 -> 185.5 mm
- net Net-(R8-Pad4): track 0.00 -> 41.0 mm, vias 0 -> 1
- net /M5V: track 77.0 -> 112.9 mm
- net Net-(R8-Pad5): track 0.00 -> 32.7 mm
- net Net-(R11-Pad2): track 31.2 -> 0.00 mm
- net Net-(R8-Pad7): track 0.00 -> 30.1 mm
- net Net-(R13-Pad2): track 28.1 -> 0.00 mm, vias 1 -> 0
- net Net-(U7-Pad1): track 27.5 -> 0.00 mm
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Other:
- board text added: "BUS_BRIDGE_ENCODERS_SHAFT REV. B 3OCT2014 (C) GRAMLICH"
- board text added: "RESET"
- board text removed: "BUS_BRIDGE_ENCODERS_SHAFT REV. A 12AUG2014 (c) GRAMLICH"
