File: rev_b/bus_bridge_encoders_sonar.sch (KiCad schematic (older format))
At the start: 63 parts, among them J1 POWER_SELECT, J2 TERMINATE_JUMPER, SW1 MJTP1243, U1 LM2940, U2 LTV-826, U3 LTV-826, U4 LTV-826, U5 754410, U6 LM2940, U7 74HCT08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

Commit message: Did first cut of revision B.
Parts:
- removed N3, N4: ENCODER_CONNECTOR, symbol ENCODER_CONNECTOR
- removed N5, N6: MOTOR_CONNECTOR, symbol MOTOR_CONNECTOR
- removed R10, R11, R12, R13, R8, R9: 10K, symbol R_VERT
- removed R2, R3, R4, R5, R6, R7: 470, symbol R_HORIZ
- removed R21: 33K, symbol R_VERT
- added D2: LED, symbol LED
- added N3: AVR_ISP_HEADER, Bus_Bridge_Encoders_Sonar:Pin_Header_Straight_2x03, symbol AVR_ISP_HEADER
- added N5, N6: MOTOR_ENCODER_CONN, Bus_Bridge_Encoders_Sonar:Pin_Header_Straight_2x04_Shrouded, symbol MOTOR_ENCODER_CONN
- added R2: 470, Bus_Bridge_Encoders_Sonar:DIP-16__300, symbol R_HORIZ_DIP16
- added R8: 10K, Bus_Bridge_Encoders_Sonar:Pin_Header_Straight_1x07, symbol R_VERT_SIP7
- added unit 3 of U7
- added unit 4 of U7
- C1, C3, C6, C9: footprint (none) -> Bus_Bridge_Encoders_Sonar:Capacitor4x3RM2-5_RevB
- C10, C11, C12, C13, C14, C2, C4, C5, C7, C8: footprint (none) -> Bus_Bridge_Encoders_Sonar:Capacitor3MMDiscRM2.5
- D1: footprint (none) -> Bus_Bridge_Encoders_Sonar:Diode_DO-41_SOD81_Horizontal_RM10
- G1: footprint (none) -> Bus_Bridge_Encoders_Sonar:OSHW_LOGO_300mil
- H1, H2, H3, H4: footprint (none) -> Bus_Bridge_Encoders_Sonar:MountingHole_3mm
- J1, J2: footprint (none) -> Bus_Bridge_Encoders_Sonar:Pin_Header_Straight_1x03
- N1: footprint (none) -> Bus_Bridge_Encoders_Sonar:Pin_Header_Straight_2x05_Shrouded
- N2: footprint (none) -> Bus_Bridge_Encoders_Sonar:Pin_Header_Straight_1x06
- N7, N8: footprint (none) -> Bus_Bridge_Encoders_Sonar:Pin_Header_Straight_1x04
- R1, R14, R15, R16, R19, R22: footprint (none) -> Bus_Bridge_Encoders_Sonar:Resistor_Horizontal_400
- R17, R20: value 22K -> 100K; footprint (none) -> Bus_Bridge_Encoders_Sonar:Resistor_Horizontal_400
- R18: value 33K -> 100K; footprint (none) -> Bus_Bridge_Encoders_Sonar:Resistor_Horizontal_400
- SW1: footprint (none) -> Bus_Bridge_Encoders_Sonar:Button_6.5MM
- U1, U6: footprint (none) -> Bus_Bridge_Encoders_Sonar:TO-220_Neutral123_Horizontal_LargePads
- U2, U3, U4, U8: footprint (none) -> Bus_Bridge_Encoders_Sonar:DIP-8__300
- U5: footprint (none) -> Bus_Bridge_Encoders_Sonar:DIP-16__300
- U7: footprint (none) -> Bus_Bridge_Encoders_Sonar:DIP-14__300
- U9: footprint (none) -> Bus_Bridge_Encoders_Sonar:DIP-28__300
- X1: footprint (none) -> Bus_Bridge_Encoders_Sonar:Crystal_HC49-U_Vertical
Connections:
- net +5V: now also R18.2, N3.2 (5V), N5.8 (VCC), N6.8 (VCC), U7.12, U7.13, U7.14 (VCC), U7.14 (VCC)
- net A0: now also N5.1 (QUAD_A); no longer N8.2 (ECHO)
- net A1: now also N5.7 (QUAD_B); no longer N7.2 (ECHO)
- net BGND: now also R8.1, R8.1, R8.1, R8.1, R8.1, R8.1
- net D10: now also R2.1 (A)
- net D11: now also N3.4 (MOSI), R2.3 (A)
- net D12: now also N3.1 (MISO), R2.2 (A)
- net D13: now also N3.3 (SCK), R2.4 (A)
- net D2: now also N6.1 (QUAD_A)
- net D3: now also N8.2 (ECHO); no longer N8.3 (TRIG)
- net D4: now also N8.3 (TRIG)
- net D5: now also N7.3 (TRIG)
- net D6: now also N7.2 (ECHO)
- net D7: now also N6.7 (QUAD_B)
- net D8: now also R2.6 (A)
- net D9: now also R2.5 (A); no longer N7.3 (TRIG)
- net GND: now also D2.-, N3.6 (GND), N5.2 (LGND), N6.2 (LGND), U7.7 (GND), U7.7 (GND); no longer R18.1
- net M1+: now also N6.3 (MOTOR_A), N6.4 (MOTOR_A)
- net M1-: now also N6.5 (MOTOR_B), N6.6 (MOTOR_B)
- net M2+: now also N5.3 (MOTOR_A), N5.4 (MOTOR_A)
- net M2-: now also N5.5 (MOTOR_B), N5.6 (MOTOR_B)
- net TXD: now also U8.1 (TXD); no longer U8.4 (RXD)
- net ~RESET: now also N3.5 (#RESET)
- net at U2.3: now also R2.15 (B)
- net at U2.5, U5.1 (EN12): now also R8.6
- net at U3.3: now also R2.13 (B)
- net at U3.5, U5.10 (3A): now also R8.4
- net at U4.1: now also R2.12 (B)
- net at U4.7, U5.9 (EN34): now also R8.3
- net at U4.3: now also R2.11 (B)
- net at U4.5, U5.15 (4A): now also R8.2
- net at U2.1: now also R2.16 (B)
- net at U2.7, U5.2 (1A): now also R8.7
- net at U3.1: now also R2.14 (B)
- net at U3.7, U5.7 (2A): now also R8.5
- net at U9.28 (PC5/ADC5/SCL): now also R2.10 (B)
- net at U7.1: now also R18.1, U8.4 (RXD); no longer U8.1 (TXD)
- net at N2.4 (TXD), R17.1, U7.2: no longer R18.2
- new net: U7.10, U7.11, U7.9
- new net: D2.+, R2.7 (A)
Other:
- note added: "Electrically\nIsolated"
- moved on the sheet: C4, G1, H1, H2, H3, H4, N7, N8, U2B, U3A, U3B, U4A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

Commit message: Rev. B is done.
Parts:
- D2: footprint (none) -> Bus_Bridge_Encoders_Sonar:T1_LED
- R2: value 470 -> 470_DIP16
- R8: value 10K -> 10Kx6
Other:
- moved on the sheet: R8A, R8B, R8C, R8D, R8E
Changed lines of the file:
@@
 P 7100 5900
 F 0 "R8" H 7145 5970 50  0000 L CNN
-F 1 "10K" H 7145 5870 50  0000 L CNN
+F 1 "10Kx6" H 7145 5870 50  0000 L CNN
 F 2 "Bus_Bridge_Encoders_Sonar:Pin_Header_Straight_1x07" H 7100 5900 50  0001 C CNN
 F 3 "" H 7100 5900 50  0000 C CNN
@@
 L R_VERT_SIP7 R8
 U 5 1 542D6F2D
-P 7400 5900
-F 0 "R8" H 7445 5970 50  0000 L CNN
-F 1 "10K" H 7445 5870 50  0000 L CNN
-F 2 "Bus_Bridge_Encoders_Sonar:Pin_Header_Straight_1x07" H 7400 5900 50  0001 C CNN
-F 3 "" H 7400 5900 50  0000 C CNN
-	5    7400 5900
+P 7500 5900
+F 0 "R8" H 7545 5970 50  0000 L CNN
+F 1 "10Kx6" H 7545 5870 50  0000 L CNN
+F 2 "Bus_Bridge_Encoders_Sonar:Pin_Header_Straight_1x07" H 7500 5900 50  0001 C CNN
+F 3 "" H 7500 5900 50  0000 C CNN
+	5    7500 5900
 	1    0    0    -1
 $EndComp
@@
 L R_VERT_SIP7 R8
 U 4 1 542D6F99
-P 7700 5900
-F 0 "R8" H 7745 5970 50  0000 L CNN
-F 1 "10K" H 7745 5870 50  0000 L CNN
-F 2 "Bus_Bridge_Encoders_Sonar:Pin_Header_Straight_1x07" H 7700 5900 50  0001 C CNN
-F 3 "" H 7700 5900 50  0000 C CNN
-	4    7700 5900
+P 7900 5900
+F 0 "R8" H 7945 5970 50  0000 L CNN
+F 1 "10Kx6" H 7945 5870 50  0000 L CNN
+F 2 "Bus_Bridge_Encoders_Sonar:Pin_Header_Straight_1x07" H 7900 5900 50  0001 C CNN
+F 3 "" H 7900 5900 50  0000 C CNN
+	4    7900 5900
 	1    0    0    -1
 $EndComp
@@
 L R_VERT_SIP7 R8
 U 3 1 542D6FFA
-P 8000 5900
-F 0 "R8" H 8045 5970 50  0000 L CNN
-F 1 "10K" H 8045 5870 50  0000 L CNN
-F 2 "Bus_Bridge_Encoders_Sonar:Pin_Header_Straight_1x07" H 8000 5900 50  0001 C CNN
-F 3 "" H 8000 5900 50  0000 C CNN
-	3    8000 5900
+P 8300 5900
+F 0 "R8" H 8345 5970 50  0000 L CNN
+F 1 "10Kx6" H 8345 5870 50  0000 L CNN
+F 2 "Bus_Bridge_Encoders_Sonar:Pin_Header_Straight_1x07" H 8300 5900 50  0001 C CNN
+F 3 "" H 8300 5900 50  0000 C CNN
+	3    8300 5900
 	1    0    0    -1
 $EndComp
@@
 L R_VERT_SIP7 R8
 U 2 1 542D7058
-P 8300 5900
-F 0 "R8" H 8345 5970 50  0000 L CNN
-F 1 "10K" H 8345 5870 50  0000 L CNN
-F 2 "Bus_Bridge_Encoders_Sonar:Pin_Header_Straight_1x07" H 8300 5900 50  0001 C CNN
-F 3 "" H 8300 5900 50  0000 C CNN
-	2    8300 5900
+P 8300 5200
+F 0 "R8" H 8345 5270 50  0000 L CNN
+F 1 "10Kx6" H 8345 5170 50  0000 L CNN
+F 2 "Bus_Bridge_Encoders_Sonar:Pin_Header_Straight_1x07" H 8300 5200 50  0001 C CNN
+F 3 "" H 8300 5200 50  0000 C CNN
+	2    8300 5200
 	1    0    0    -1
 $EndComp
@@
 L R_VERT_SIP7 R8
 U 1 1 542D70C3
-P 8600 5900
-F 0 "R8" H 8645 5970 50  0000 L CNN
-F 1 "10K" H 8645 5870 50  0000 L CNN
-F 2 "Bus_Bridge_Encoders_Sonar:Pin_Header_Straight_1x07" H 8600 5900 50  0001 C CNN
-F 3 "" H 8600 5900 50  0000 C CNN
-	1    8600 5900
+P 8400 4350
+F 0 "R8" H 8445 4420 50  0000 L CNN
+F 1 "10Kx6" H 8445 4320 50  0000 L CNN
+F 2 "Bus_Bridge_Encoders_Sonar:Pin_Header_Straight_1x07" H 8400 4350 50  0001 C CNN
+F 3 "" H 8400 4350 50  0000 C CNN
+	1    8400 4350
 	1    0    0    -1
 $EndComp
@@
 	7700 800  5700 800
 Wire Wire Line
-	7800 1400 7800 5300
+	7800 1400 7800 5400
 Connection ~ 7600 1200
 Connection ~ 7600 700
@@
 Connection ~ 7900 2300
 Wire Wire Line
-	7400 5600 7400 5700
+	7500 5500 7500 5700
 Connection ~ 8000 3000
 Connection ~ 8100 3700
 Wire Wire Line
-	8100 5600 8000 5600
-Wire Wire Line
-	8000 5600 8000 5700
-Connection ~ 8200 4400
-Connection ~ 8300 5100
-Wire Wire Line
-	7100 5500 7100 5700
+	7100 5400 7100 5700
 Wire Wire Line
 	7100 6200 7100 6100
@@
 	7900 2300 7500 2300
 Wire Wire Line
-	7900 1500 7900 5400
+	7900 1500 7900 5500
 Wire Wire Line
 	8400 1500 7900 1500
@@
 	8000 3000 7500 3000
 Wire Wire Line
-	8000 1600 8000 5500
+	8000 1600 8000 5600
 Wire Wire Line
 	8100 3700 7500 3700
 Wire Wire Line
-	8100 1800 8100 5600
-Wire Wire Line
 	8600 1800 8100 1800
-Wire Wire Line
-	8200 4400 7500 4400
-Wire Wire Line
-	8200 2000 8200 5600
-Wire Wire Line
-	7500 5100 8300 5100
-Wire Wire Line
-	8300 2200 8300 5500
 Wire Wire Line
 	5200 600  9700 600
@@
 Connection ~ 9700 2500
 Wire Wire Line
-	7700 2700 9700 2700
+	9700 2700 7700 2700
 Wire Wire Line
 	9700 2500 9600 2500
 Wire Wire Line
-	9700 2700 9700 2400
+	9700 2400 9700 2700
 Wire Wire Line
 	9700 2400 9600 2400
-Connection ~ 7400 6200
-Connection ~ 7700 6200
-Wire Wire Line
-	7400 6200 7400 6100
-Connection ~ 8000 6200
-Wire Wire Line
-	7700 6200 7700 6100
+Connection ~ 7500 6200
+Connection ~ 7900 6200
+Wire Wire Line
+	7500 6200 7500 6100
 Connection ~ 8300 6200
 Wire Wire Line
-	8000 6200 8000 6100
+	7900 6200 7900 6100
 Wire Wire Line
 	8300 6200 8300 6100
 Wire Wire Line
-	7000 6200 8600 6200
-Wire Wire Line
-	8600 6200 8600 6100
+	8700 6200 7000 6200
 Connection ~ 5400 2200
 Wire Wire Line
@@
 	2600 3500 2000 3500
 Wire Wire Line
-	2000 3500 2000 4450
-Wire Wire Line
-	2000 4450 1700 4450
+	2000 4450 2000 3500
+Wire Wire Line
+	1700 4450 2000 4450
 Wire Wire Line
 	1100 4450 1000 4450
@@
 	9900 5450 9850 5450
 Wire Wire Line
-	7000 5400 7000 6200
+	7000 6200 7000 5300
 Connection ~ 7100 6200
 Connection ~ 7700 2700
@@
 	9800 2800 8600 2800
 Wire Wire Line
-	8600 2800 8600 5300
-Wire Wire Line
-	8600 5300 9200 5300
-Wire Wire Line
 	9100 5300 9100 5400
 Wire Wire Line
@@
 Connection ~ 9100 5300
 Wire Wire Line
-	8700 5200 9200 5200
-Wire Wire Line
 	9100 5200 9100 5100
 Wire Wire Line
@@
 	9400 3700 9400 3800
 Connection ~ 9400 3800
-Wire Wire Line
-	8300 5600 8300 5700
-Wire Wire Line
-	8200 5600 8300 5600
-Wire Wire Line
-	8300 5500 8600 5500
-Wire Wire Line
-	8600 5500 8600 5700
 Wire Wire Line
 	9000 4600 10400 4600
@@
 	9000 5500 9000 6300
 Wire Wire Line
-	7000 5400 7400 5400
-Wire Wire Line
-	7700 800  7700 5200
-Wire Wire Line
-	7100 5500 7500 5500
-Wire Wire Line
-	7600 5600 7400 5600
+	7700 5300 7000 5300
+Wire Wire Line
+	7700 800  7700 5300
+Wire Wire Line
+	7800 5400 7100 5400
+Wire Wire Line
+	7900 5500 7500 5500
 Wire Notes Line
 	9150 5450 8850 5450
@@
 Wire Notes Line
 	8850 6250 6950 6250
-Wire Wire Line
-	7700 5700 7700 5600
-Wire Wire Line
-	7700 5600 7900 5600
-Wire Wire Line
-	7900 5600 7900 5500
-Wire Wire Line
-	7900 5500 8000 5500
-Wire Wire Line
-	7600 5600 7600 5500
-Wire Wire Line
-	7600 5500 7800 5500
-Wire Wire Line
-	7800 5500 7800 5400
-Wire Wire Line
-	7800 5400 7900 5400
-Wire Wire Line
-	7500 5500 7500 5400
-Wire Wire Line
-	7500 5400 7700 5400
-Wire Wire Line
-	7700 5400 7700 5300
-Wire Wire Line
-	7700 5300 7800 5300
-Wire Wire Line
-	7400 5400 7400 5300
-Wire Wire Line
-	7400 5300 7600 5300
-Wire Wire Line
-	7600 5300 7600 5200
-Wire Wire Line
-	7600 5200 7700 5200
 Wire Notes Line
 	6950 6250 6950 5300
-Wire Wire Line
-	8700 2900 8700 5200
 Connection ~ 9100 5200
 Connection ~ 1700 3000
@@
 P 5800 2600
 F 0 "R2" H 5800 2700 50  0000 C CNN
-F 1 "470" H 5800 2500 50  0000 C CNN
+F 1 "470_DIP16" H 5800 2500 50  0000 C CNN
 F 2 "Bus_Bridge_Encoders_Sonar:DIP-16__300" H 5825 2600 60  0001 C CNN
 F 3 "" H 5825 2600 60  0000 C CNN
@@
 P 5800 2900
 F 0 "R2" H 5800 3000 50  0000 C CNN
-F 1 "470" H 5800 2800 50  0000 C CNN
+F 1 "470_DIP16" H 5800 2800 50  0000 C CNN
 F 2 "Bus_Bridge_Encoders_Sonar:DIP-16__300" H 5825 2900 60  0001 C CNN
 F 3 "" H 5825 2900 60  0000 C CNN
@@
 P 5800 3200
 F 0 "R2" H 5800 3300 50  0000 C CNN
-F 1 "470" H 5800 3100 50  0000 C CNN
+F 1 "470_DIP16" H 5800 3100 50  0000 C CNN
 F 2 "Bus_Bridge_Encoders_Sonar:DIP-16__300" H 5825 3200 60  0001 C CNN
 F 3 "" H 5825 3200 60  0000 C CNN
@@
 P 5800 3500
 F 0 "R2" H 5800 3600 50  0000 C CNN
-F 1 "470" H 5800 3400 50  0000 C CNN
+F 1 "470_DIP16" H 5800 3400 50  0000 C CNN
 F 2 "Bus_Bridge_Encoders_Sonar:DIP-16__300" H 5825 3500 60  0001 C CNN
 F 3 "" H 5825 3500 60  0000 C CNN
@@
 P 5800 3900
 F 0 "R2" H 5800 4000 50  0000 C CNN
-F 1 "470" H 5800 3800 50  0000 C CNN
+F 1 "470_DIP16" H 5800 3800 50  0000 C CNN
 F 2 "Bus_Bridge_Encoders_Sonar:DIP-16__300" H 5825 3900 60  0001 C CNN
 F 3 "" H 5825 3900 60  0000 C CNN
@@
 P 5800 4200
 F 0 "R2" H 5800 4300 50  0000 C CNN
-F 1 "470" H 5800 4100 50  0000 C CNN
+F 1 "470_DIP16" H 5800 4100 50  0000 C CNN
 F 2 "Bus_Bridge_Encoders_Sonar:DIP-16__300" H 5825 4200 60  0001 C CNN
 F 3 "" H 5825 4200 60  0000 C CNN
@@
 F 0 "D2" H 4370 5810 50  0000 C CNN
 F 1 "LED" H 4410 5525 50  0000 C CNN
-F 2 "" H 4300 5650 60  0000 C CNN
+F 2 "Bus_Bridge_Encoders_Sonar:T1_LED" H 4300 5650 60  0001 C CNN
 F 3 "" H 4300 5650 60  0000 C CNN
 	1    4300 5650
@@
 P 4600 5300
 F 0 "R2" H 4600 5400 50  0000 C CNN
-F 1 "470" H 4600 5200 50  0000 C CNN
+F 1 "470_DIP16" H 4600 5200 50  0000 C CNN
 F 2 "Bus_Bridge_Encoders_Sonar:DIP-16__300" H 4625 5300 60  0001 C CNN
 F 3 "" H 4625 5300 60  0000 C CNN
@@
 Wire Wire Line
 	4300 5900 4300 6000
+Wire Wire Line
+	8900 5200 9200 5200
+Wire Wire Line
+	8900 5200 8900 4000
+Wire Wire Line
+	8900 4000 8700 4000
+Wire Wire Line
+	8700 4000 8700 2900
+Wire Wire Line
+	8800 5300 9200 5300
+Wire Wire Line
+	8800 5300 8800 4100
+Wire Wire Line
+	8800 4100 8600 4100
+Wire Wire Line
+	8600 4100 8600 2800
+Wire Wire Line
+	8400 4000 8400 4150
+Wire Wire Line
+	8400 4550 8400 4800
+Wire Wire Line
+	8400 4800 8700 4800
+Wire Wire Line
+	8700 4800 8700 6200
+Connection ~ 8300 4000
+Wire Wire Line
+	7500 5100 7600 5100
+Wire Wire Line
+	7600 5100 7600 4800
+Wire Wire Line
+	8300 4800 7600 4800
+Wire Wire Line
+	8400 4000 8300 4000
+Wire Wire Line
+	7500 4400 8200 4400
+Connection ~ 8200 4400
+Wire Wire Line
+	8300 5000 8300 4900
+Wire Wire Line
+	8200 4900 8300 4900
+Wire Wire Line
+	8200 2000 8200 4900
+Wire Wire Line
+	8300 5400 8300 5500
+Wire Wire Line
+	8300 5500 8700 5500
+Connection ~ 8700 5500
+Wire Wire Line
+	8300 5700 8300 5600
+Wire Wire Line
+	8100 5600 8300 5600
+Wire Wire Line
+	8100 1800 8100 5600
+Wire Wire Line
+	8300 2200 8300 4800
+Wire Wire Line
+	8000 5600 7900 5600
+Wire Wire Line
+	7900 5600 7900 5700
 $EndSCHEMATC
