File: rev_d/$power.sch (KiCad schematic (older format))
At the start: 15 parts, among them J1 POWER_SELECT, Q1 PN2222, U1 LTV-826, U2 LTV-826, U3 LTV-826, U4 LTV-826, U5 LM2940, U6 754410

Commit message: Rev. D appears to be ready.
Parts:
- R1, R2: footprint Bus_Bridge_Encoders_Sonar:Pin_Header_Straight_1x02 -> Bus_Bridge_Encoders_Sonar:Resistor_Vertical__100
Changed lines of the file:
@@
 F 0 "R1" H 2650 7500 50  0000 C CNN
 F 1 ".47" H 2650 7300 50  0000 C CNN
-F 2 "Bus_Bridge_Encoders_Sonar:Pin_Header_Straight_1x02" H 2675 7400 60  0001 C CNN
+F 2 "Bus_Bridge_Encoders_Sonar:Resistor_Vertical__100" H 2675 7400 60  0001 C CNN
 F 3 "" H 2675 7400 60  0000 C CNN
 	1    2650 7400
@@
 F 0 "R2" H 3170 5950 50  0000 L CNN
 F 1 "220" H 3170 5850 50  0000 L CNN
-F 2 "Bus_Bridge_Encoders_Sonar:Pin_Header_Straight_1x02" H 3100 5950 60  0001 C CNN
+F 2 "Bus_Bridge_Encoders_Sonar:Resistor_Vertical__100" H 3100 5950 60  0001 C CNN
 F 3 "" H 3100 5950 60  0000 C CNN
 	1    3100 5900
