File: rev_d/bus_bridge_encoders_sonar.kicad_pcb (KiCad board)
At the start: 2 copper layers, 100 x 50 mm, 61 parts, among them J1 POWER_SELECT, J2 TERMINATE_JUMPER, Q1 PN2222, Q2 PN2222, Q3 PN2222, Q4 PN2222, Q5 PN2222, SW1 MJTP1243, U1 LTV-826, U10 ATMEGA328_DIP28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

Commit message: Rev. D appears to be ready.
Parts:
- C13: value .1uF -> 1uF
- R4: value .47 -> 120
- moved J1 5.72 mm to (198.1, 128.3)
- moved N5 2.54 mm to (141.0, 125.7)
- moved C2 2.54 mm to (194.9, 127.0)
- moved C3 2.54 mm to (194.9, 132.7)
- moved C1 2.01 mm to (196.2, 139.1), turned to 180 degrees
- moved U7 1.27 mm to (140.3, 113.0)
- moved C12 0.64 mm to (140.3, 101.6)
- moved R10 0.63 mm to (132.1, 118.7)
- moved R9 0.63 mm to (132.1, 114.9)
- moved R1 0.13 mm to (191.1, 127.0)
Connections:
- net VCC renamed +5V
- N1 pad 10: /Power/BGND -> /Power/BPWR
- N1 pad 7: /Power/BPWR -> /Power/BGND
- N1 pad 8: /Power/BPWR -> /Power/BGND
- N1 pad 9: /Power/BGND -> /Power/BPWR
Routing:
- net GND: track 412.4 -> 443.5 mm, vias 28 -> 32
- net /Power/BPWR: track 131.8 -> 138.8 mm
- net /Power/MOTOR_POWER: track 16.9 -> 10.7 mm
- net /Power/LED_5V: track 147.9 -> 142.2 mm
- net /Logic/~RESET: track 84.8 -> 81.1 mm
- net /Logic/D13: track 42.9 -> 46.3 mm
- net /Logic/D12: track 22.5 -> 20.1 mm
- net /Logic/D11: track 20.0 -> 18.1 mm, vias 1 -> 0
- net Net-(R10-Pad1): track 44.8 -> 46.6 mm
- net +5V: track 257.3 -> 255.7 mm, vias 3 -> 4
- net Net-(C13-Pad1): track 16.7 -> 15.4 mm
- net Net-(N4-Pad6): track 50.9 -> 52.1 mm
- net /Power/MOTOR1_B: track 36.6 -> 37.6 mm
- net Net-(C2-Pad2): track 4.81 -> 3.81 mm
- net /Logic/CANL: track 21.4 -> 20.6 mm
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Other:
- board text added: "ISP"
- board text added: "REV. D 30OCT2014"
- board text removed: "REV. C 16OCT2014"
