File: rev_d/logic.sch (KiCad schematic (older format))
At the start: 43 parts, among them J2 TERMINATE_JUMPER, Q2 PN2222, Q3 PN2222, Q4 PN2222, Q5 PN2222, SW1 MJTP1243, U10 ATMEGA328_DIP28, U7 74HCT08, U8 LM2940, U9 MCP2562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

Commit message: Rev. D appears to be ready.
Parts:
- C13: value .1uF -> 1uF
- R4: value .47 -> 120
Other:
- note added: "+"
- note added: "35V\nAluminum"
- note added: "6.3V\nTantalum"
Changed lines of the file:
@@
 encoding utf-8
 Sheet 3 3
-Title ""
-Date "Sun 12 Oct 2014"
-Rev "C"
+Title "Bus Bridge/Encoders/Sonars"
+Date "Thu 30 Oct 2014"
+Rev "D"
 Comp ""
 Comment1 ""
@@
 P 1500 3950
 F 0 "R4" H 1500 4050 50  0000 C CNN
-F 1 ".47" H 1500 3850 50  0000 C CNN
+F 1 "120" H 1500 3850 50  0000 C CNN
 F 2 "Bus_Bridge_Encoders_Sonar:Pin_Header_Straight_1x02" H 1525 3950 60  0001 C CNN
 F 3 "" H 1525 3950 60  0000 C CNN
@@
 P 4100 5300
 F 0 "C13" H 4160 5360 50  0000 L CNN
-F 1 ".1uF" H 4160 5230 50  0000 L CNN
+F 1 "1uF" H 4160 5230 50  0000 L CNN
 F 2 "Bus_Bridge_Encoders_Sonar:Capacitor4x3RM2-5_RevB" H 4138 5150 30  0001 C CNN
 F 3 "" H 4100 5300 60  0000 C CNN
@@
 	4250 6950 4250 7050
 Connection ~ 3950 6950
+Text Notes 1400 7400 0    50   ~ 0
+35V\nAluminum
+Text Notes 1250 7050 0    50   ~ 0
++
+Text Notes 2650 7050 0    50   ~ 0
++
+Text Notes 2800 7400 0    50   ~ 0
+6.3V\nTantalum
 $EndSCHEMATC

Commit message: Split 22uF Capacitors into Aluminum and Tantalum.
Parts:
- C5: value 22uF -> 22uF_35V_ALUM
- C8: value 22uF -> 22uF_6.3V_TANT
- R10, R11, R4, R5, R6, R7, R8, R9: footprint Bus_Bridge_Encoders_Sonar:Pin_Header_Straight_1x02 -> Bus_Bridge_Encoders_Sonar:Resistor_Vertical__100
- R12: value 4K7x4 -> 4K7_SIP5
Other:
- moved on the sheet: C11, C12, C14, C6, C8, C9, G1, R8, U8
